File: Development Board/CanSat.kicad_pcb (KiCad board)
At the start: 2 copper layers, 100 x 60 mm, 21 parts, among them J1 Screw_Terminal_01x02, U1 Pico, U2 L7805

Commit message: Add files via upload
Parts:
- added G***: LOGO, Logo:logo, F.Cu at (171.9, 102.7)
- added G***: LOGO, Logo:logo, F.Cu at (409.9, 27.7)
- moved GPS1 10.2 mm to (148.9, 120.7), turned to 0 degrees
- moved BMP280 10.1 mm to (124.2, 120.8), turned to 0 degrees
Routing:
- net +5V: track 153.8 -> 178.3 mm
- net /RXD: track 60.4 -> 73.0 mm, vias 0 -> 2
- net GND: track 236.6 -> 229.1 mm
- net /SDA: track 92.2 -> 96.6 mm, vias 1 -> 2
- net /TXD: track 68.8 -> 72.6 mm
- net /RST: track 44.3 -> 45.2 mm
- net /SCL: track 73.3 -> 73.8 mm, vias 2 -> 1
Other:
- board text added: "CanSat"
- board text added: "CanSat Development Board v1"
- board text added: "Pico"
- board text removed: "CanSat Development Board"
